File: rf_split/v1_rev-/active_rf_split_4way.kicad_pcb (KiCad board)
At the start: 2 copper layers, 28.6 x 31.8 mm, 34 parts, among them J0 RF_IN, J1 OUT1, J2 OUT2, J3 OUT3, J4 OUT4, U1 BGA2815, U2 LP2985-3.3

Commit message: updated rf amp decoupling capacitor value
Parts:
- C1: value 0.01uF -> 470pF
