File: noise_switch/v2_rev-/noise_switch.sch (KiCad schematic (older format))
At the start: 24 parts, among them J1 RCVR, J2 ANT, J3 NOISE, U1 74LVC2G06, U2 MASWSS0176

Commit message: adding pdf of schematic
Other:
- note added: "C2, C3, C4, C6, C7: \n1000 pF for 100 MHz - 1 GHz\n39 pF for 0.5 GHz - 3 GHz"
- note removed: "C6,C7: \n1000 pF for 100 MHz - 1 GHz\n39 pF for 0.5 GHz - 3 GHz"
- moved on the sheet: C1, C2, C3, C4, C5, C6, C7, H1, H2, H3, J1, J2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
